File: light-pattern/light-pattern.sch (KiCad schematic (older format))
At the start: 28 parts

Commit message: updated schematic
Parts:
- R4, R6: value 1K -> 10K
- R5: value 1K -> 330
Changed lines of the file:
@@
 P 7750 4150
 F 0 "R4" V 7650 4100 50  0000 L CNN
-F 1 "1K" V 7850 4100 50  0000 L CNN
+F 1 "10K" V 7850 4100 50  0000 L CNN
 F 2 "" H 7750 4150 50  0001 C CNN
 F 3 "~" H 7750 4150 50  0001 C CNN
@@
 P 8150 4150
 F 0 "R5" V 8050 4100 50  0000 L CNN
-F 1 "1K" V 8250 4100 50  0000 L CNN
+F 1 "330" V 8250 4100 50  0000 L CNN
 F 2 "" H 8150 4150 50  0001 C CNN
 F 3 "~" H 8150 4150 50  0001 C CNN
@@
 P 8550 4150
 F 0 "R6" V 8450 4100 50  0000 L CNN
-F 1 "1K" V 8650 4100 50  0000 L CNN
+F 1 "10K" V 8650 4100 50  0000 L CNN
 F 2 "" H 8550 4150 50  0001 C CNN
 F 3 "~" H 8550 4150 50  0001 C CNN

Commit message: Removed power switch from Arduino
Parts:
- removed POWER: SW_Push, symbol Switch:SW_Push
- renumbered sw_all to sw_triggerAll, sw_decr to sw_triggerDown, sw_rand to sw_triggerRandom, sw_incr to sw_triggerUp
Connections:
- net VCC: now also Arduino_UNO_R2.5 (+5V), sw_triggerAll.2, sw_triggerDown.2, sw_triggerRandom.2, sw_triggerUp.2
Changed lines of the file:
@@
 L power:VCC #PWR?
 U 1 1 614C4F7D
-P 3450 2550
-F 0 "#PWR?" H 3450 2400 50  0001 C CNN
-F 1 "VCC" H 3465 2723 50  0000 C CNN
-F 2 "" H 3450 2550 50  0001 C CNN
-F 3 "" H 3450 2550 50  0001 C CNN
-	1    3450 2550
+P 3450 3100
+F 0 "#PWR?" H 3450 2950 50  0001 C CNN
+F 1 "VCC" H 3465 3273 50  0000 C CNN
+F 2 "" H 3450 3100 50  0001 C CNN
+F 3 "" H 3450 3100 50  0001 C CNN
+	1    3450 3100
 	1    0    0    -1
 $EndComp
@@
 Wire Wire Line
 	3250 5500 3250 5650
-$Comp
-L Switch:SW_Push POWER
-U 1 1 61514A08
-P 3450 2900
-F 0 "POWER" H 3600 2800 50  0000 R CNN
-F 1 "SW_Push" H 3450 3094 50  0001 C CNN
-F 2 "" H 3450 3100 50  0001 C CNN
-F 3 "~" H 3450 3100 50  0001 C CNN
-	1    3450 2900
-	0    -1   -1   0
-$EndComp
-Wire Wire Line
-	3450 2550 3450 2700
 Wire Wire Line
 	3450 3200 3450 3100
@@
 	4500 4300 4500 4150
 $Comp
-L Switch:SW_Push sw_incr
+L Switch:SW_Push sw_triggerUp
 U 1 1 61532EBA
 P 4950 3550
-F 0 "sw_incr" H 4950 3500 50  0000 C CNN
+F 0 "sw_triggerUp" H 4950 3500 50  0000 C CNN
 F 1 "SW_Push" H 4950 3744 50  0001 C CNN
 F 2 "" H 4950 3750 50  0001 C CNN
@@
 	4500 3750 4500 3850
 $Comp
-L Switch:SW_Push sw_decr
+L Switch:SW_Push sw_triggerDown
 U 1 1 61533F79
 P 5400 3550
-F 0 "sw_decr" H 5400 3500 50  0000 C CNN
+F 0 "sw_triggerDown" H 5400 3500 50  0000 C CNN
 F 1 "SW_Push" H 5400 3744 50  0001 C CNN
 F 2 "" H 5400 3750 50  0001 C CNN
@@
 $EndComp
 $Comp
-L Switch:SW_Push sw_rand
+L Switch:SW_Push sw_triggerRandom
 U 1 1 615362EE
 P 5850 3550
-F 0 "sw_rand" H 5850 3500 50  0000 C CNN
+F 0 "sw_triggerRandom" H 5850 3500 50  0000 C CNN
 F 1 "SW_Push" H 5850 3744 50  0001 C CNN
 F 2 "" H 5850 3750 50  0001 C CNN
@@
 	5850 3850 5850 3950
 $Comp
-L Switch:SW_Push sw_all
+L Switch:SW_Push sw_triggerAll
 U 1 1 614AAAD7
 P 4500 3550
-F 0 "sw_all" H 4500 3500 50  0000 C CNN
+F 0 "sw_triggerAll" H 4500 3500 50  0000 C CNN
 F 1 "SW_Push" H 4500 3744 50  0001 C CNN
 F 2 "" H 4500 3750 50  0001 C CNN

Commit message: Updated schematic diagram
Parts:
- renumbered sw_triggerAll to sw_triggerAll1, sw_triggerDown to sw_triggerDown1, sw_triggerRandom to sw_triggerRandom1, sw_triggerUp to sw_triggerUp1
Connections:
- net A_D2: no longer led9.2 (A)
- net A_D10: now reaches Arduino_UNO_R2.25 (D10)
- net A_D10: now also led9.2 (A)
- net VCC: no longer names the net of Arduino_UNO_R2.5 (+5V), sw_triggerAll1.2, sw_triggerDown1.2, sw_triggerRandom1.2, sw_triggerUp1.2
- no-connect marks 0 -> 12
Other:
- note added: "LED ARRAY"
- note added: "SWITCH CONTROL"
- moved on the sheet: Arduino_UNO_R2, R1, R2, R3, R4, R5, R6, R7, R8, R9, R_SW1, R_SW2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

Commit message: Updated schematic diagram
Parts:
- R1, R2, R3, R4, R5, R6, R7, R8, R9: footprint (none) -> Resistor_THT:R_Axial_DIN0207_L6.3mm_D2.5mm_P2.54mm_Vertical
- R_SW1, R_SW2, R_SW3, R_SW4: footprint (none) -> Resistor_THT:R_Axial_DIN0207_L6.3mm_D2.5mm_P5.08mm_Vertical
- led1, led2, led3, led4, led5, led6, led7, led8, led9: footprint (none) -> LED_THT:LED_D5.0mm
- sw_triggerAll1, sw_triggerDown1, sw_triggerRandom1, sw_triggerUp1: footprint (none) -> Button_Switch_THT:SW_PUSH_6mm
Changed lines of the file:
@@
 F 0 "led4" H 2850 5800 50  0000 C CNN
 F 1 "BLU" H 2850 5600 50  0000 C CNN
-F 2 "" H 2850 5700 50  0001 C CNN
+F 2 "LED_THT:LED_D5.0mm" H 2850 5700 50  0001 C CNN
 F 3 "~" H 2850 5700 50  0001 C CNN
 	1    2850 5700
@@
 F 0 "led5" H 3250 5800 50  0000 C CNN
 F 1 "ORA" H 3250 5600 50  0000 C CNN
-F 2 "" H 3250 5700 50  0001 C CNN
+F 2 "LED_THT:LED_D5.0mm" H 3250 5700 50  0001 C CNN
 F 3 "~" H 3250 5700 50  0001 C CNN
 	1    3250 5700
@@
 F 0 "R1" V 1550 6050 50  0000 L CNN
 F 1 "1K" V 1750 6050 50  0000 L CNN
-F 2 "" H 1650 6100 50  0001 C CNN
+F 2 "Resistor_THT:R_Axial_DIN0207_L6.3mm_D2.5mm_P2.54mm_Vertical" H 1650 6100 50  0001 C CNN
 F 3 "~" H 1650 6100 50  0001 C CNN
 	1    1650 6100
@@
 F 0 "R2" V 1950 6050 50  0000 L CNN
 F 1 "220" V 2150 6050 50  0000 L CNN
-F 2 "" H 2050 6100 50  0001 C CNN
+F 2 "Resistor_THT:R_Axial_DIN0207_L6.3mm_D2.5mm_P2.54mm_Vertical" H 2050 6100 50  0001 C CNN
 F 3 "~" H 2050 6100 50  0001 C CNN
 	1    2050 6100
@@
 F 0 "R3" V 2350 6050 50  0000 L CNN
 F 1 "220" V 2550 6050 50  0000 L CNN
-F 2 "" H 2450 6100 50  0001 C CNN
+F 2 "Resistor_THT:R_Axial_DIN0207_L6.3mm_D2.5mm_P2.54mm_Vertical" H 2450 6100 50  0001 C CNN
 F 3 "~" H 2450 6100 50  0001 C CNN
 	1    2450 6100
@@
 F 0 "R4" V 2750 6050 50  0000 L CNN
 F 1 "10K" V 2950 6050 50  0000 L CNN
-F 2 "" H 2850 6100 50  0001 C CNN
+F 2 "Resistor_THT:R_Axial_DIN0207_L6.3mm_D2.5mm_P2.54mm_Vertical" H 2850 6100 50  0001 C CNN
 F 3 "~" H 2850 6100 50  0001 C CNN
 	1    2850 6100
@@
 F 0 "R5" V 3150 6050 50  0000 L CNN
 F 1 "330" V 3350 6050 50  0000 L CNN
-F 2 "" H 3250 6100 50  0001 C CNN
+F 2 "Resistor_THT:R_Axial_DIN0207_L6.3mm_D2.5mm_P2.54mm_Vertical" H 3250 6100 50  0001 C CNN
 F 3 "~" H 3250 6100 50  0001 C CNN
 	1    3250 6100
@@
 F 0 "led6" H 3650 5800 50  0000 C CNN
 F 1 "BLU" H 3650 5600 50  0000 C CNN
-F 2 "" H 3650 5700 50  0001 C CNN
+F 2 "LED_THT:LED_D5.0mm" H 3650 5700 50  0001 C CNN
 F 3 "~" H 3650 5700 50  0001 C CNN
 	1    3650 5700
@@
 F 0 "R6" V 3550 6050 50  0000 L CNN
 F 1 "10K" V 3750 6050 50  0000 L CNN
-F 2 "" H 3650 6100 50  0001 C CNN
+F 2 "Resistor_THT:R_Axial_DIN0207_L6.3mm_D2.5mm_P2.54mm_Vertical" H 3650 6100 50  0001 C CNN
 F 3 "~" H 3650 6100 50  0001 C CNN
 	1    3650 6100
@@
 F 0 "led7" H 4050 5800 50  0000 C CNN
 F 1 "GRN" H 4050 5600 50  0000 C CNN
-F 2 "" H 4050 5700 50  0001 C CNN
+F 2 "LED_THT:LED_D5.0mm" H 4050 5700 50  0001 C CNN
 F 3 "~" H 4050 5700 50  0001 C CNN
 	1    4050 5700
@@
 F 0 "led8" H 4450 5800 50  0000 C CNN
 F 1 "YLW" H 4450 5600 50  0000 C CNN
-F 2 "" H 4450 5700 50  0001 C CNN
+F 2 "LED_THT:LED_D5.0mm" H 4450 5700 50  0001 C CNN
 F 3 "~" H 4450 5700 50  0001 C CNN
 	1    4450 5700
@@
 F 0 "R7" V 3950 6050 50  0000 L CNN
 F 1 "220" V 4150 6050 50  0000 L CNN
-F 2 "" H 4050 6100 50  0001 C CNN
+F 2 "Resistor_THT:R_Axial_DIN0207_L6.3mm_D2.5mm_P2.54mm_Vertical" H 4050 6100 50  0001 C CNN
 F 3 "~" H 4050 6100 50  0001 C CNN
 	1    4050 6100
@@
 F 0 "R8" V 4350 6050 50  0000 L CNN
 F 1 "220" V 4550 6050 50  0000 L CNN
-F 2 "" H 4450 6100 50  0001 C CNN
+F 2 "Resistor_THT:R_Axial_DIN0207_L6.3mm_D2.5mm_P2.54mm_Vertical" H 4450 6100 50  0001 C CNN
 F 3 "~" H 4450 6100 50  0001 C CNN
 	1    4450 6100
@@
 F 0 "led9" H 4850 5800 50  0000 C CNN
 F 1 "RED" H 4850 5600 50  0000 C CNN
-F 2 "" H 4850 5700 50  0001 C CNN
+F 2 "LED_THT:LED_D5.0mm" H 4850 5700 50  0001 C CNN
 F 3 "~" H 4850 5700 50  0001 C CNN
 	1    4850 5700
@@
 F 0 "R9" V 4750 6050 50  0000 L CNN
 F 1 "1K" V 4950 6050 50  0000 L CNN
-F 2 "" H 4850 6100 50  0001 C CNN
+F 2 "Resistor_THT:R_Axial_DIN0207_L6.3mm_D2.5mm_P2.54mm_Vertical" H 4850 6100 50  0001 C CNN
 F 3 "~" H 4850 6100 50  0001 C CNN
 	1    4850 6100
@@
 F 0 "led1" H 1650 5800 50  0000 C CNN
 F 1 "RED" H 1650 5600 50  0000 C CNN
-F 2 "" H 1650 5700 50  0001 C CNN
+F 2 "LED_THT:LED_D5.0mm" H 1650 5700 50  0001 C CNN
 F 3 "~" H 1650 5700 50  0001 C CNN
 	1    1650 5700
@@
 F 0 "led2" H 2050 5800 50  0000 C CNN
 F 1 "YLW" H 2050 5600 50  0000 C CNN
-F 2 "" H 2050 5700 50  0001 C CNN
+F 2 "LED_THT:LED_D5.0mm" H 2050 5700 50  0001 C CNN
 F 3 "~" H 2050 5700 50  0001 C CNN
 	1    2050 5700
@@
 F 0 "led3" H 2450 5800 50  0000 C CNN
 F 1 "GRN" H 2450 5600 50  0000 C CNN
-F 2 "" H 2450 5700 50  0001 C CNN
+F 2 "LED_THT:LED_D5.0mm" H 2450 5700 50  0001 C CNN
 F 3 "~" H 2450 5700 50  0001 C CNN
 	1    2450 5700
@@
 F 0 "R_SW1" V 3450 2800 50  0000 L CNN
 F 1 "10K" V 3650 2900 50  0000 L CNN
-F 2 "" H 3550 2950 50  0001 C CNN
+F 2 "Resistor_THT:R_Axial_DIN0207_L6.3mm_D2.5mm_P5.08mm_Vertical" H 3550 2950 50  0001 C CNN
 F 3 "~" H 3550 2950 50  0001 C CNN
 	1    3550 2950
@@
 F 0 "sw_triggerUp1" H 4000 2400 50  0000 C CNN
 F 1 "SW_Push" H 4000 2644 50  0001 C CNN
-F 2 "" H 4000 2650 50  0001 C CNN
+F 2 "Button_Switch_THT:SW_PUSH_6mm" H 4000 2650 50  0001 C CNN
 F 3 "~" H 4000 2650 50  0001 C CNN
 	1    4000 2450
@@
 F 0 "R_SW2" V 3900 2800 50  0000 L CNN
 F 1 "10K" V 4100 2900 50  0000 L CNN
-F 2 "" H 4000 2950 50  0001 C CNN
+F 2 "Resistor_THT:R_Axial_DIN0207_L6.3mm_D2.5mm_P5.08mm_Vertical" H 4000 2950 50  0001 C CNN
 F 3 "~" H 4000 2950 50  0001 C CNN
 	1    4000 2950
@@
 F 0 "sw_triggerDown1" H 4450 2400 50  0000 C CNN
 F 1 "SW_Push" H 4450 2644 50  0001 C CNN
-F 2 "" H 4450 2650 50  0001 C CNN
+F 2 "Button_Switch_THT:SW_PUSH_6mm" H 4450 2650 50  0001 C CNN
 F 3 "~" H 4450 2650 50  0001 C CNN
 	1    4450 2450
@@
 F 0 "R_SW3" V 4350 2800 50  0000 L CNN
 F 1 "10K" V 4550 2900 50  0000 L CNN
-F 2 "" H 4450 2950 50  0001 C CNN
+F 2 "Resistor_THT:R_Axial_DIN0207_L6.3mm_D2.5mm_P5.08mm_Vertical" H 4450 2950 50  0001 C CNN
 F 3 "~" H 4450 2950 50  0001 C CNN
 	1    4450 2950
@@
 F 0 "sw_triggerRandom1" H 4900 2400 50  0000 C CNN
 F 1 "SW_Push" H 4900 2644 50  0001 C CNN
-F 2 "" H 4900 2650 50  0001 C CNN
+F 2 "Button_Switch_THT:SW_PUSH_6mm" H 4900 2650 50  0001 C CNN
 F 3 "~" H 4900 2650 50  0001 C CNN
 	1    4900 2450
@@
 F 0 "R_SW4" V 4800 2800 50  0000 L CNN
 F 1 "10K" V 5000 2900 50  0000 L CNN
-F 2 "" H 4900 2950 50  0001 C CNN
+F 2 "Resistor_THT:R_Axial_DIN0207_L6.3mm_D2.5mm_P5.08mm_Vertical" H 4900 2950 50  0001 C CNN
 F 3 "~" H 4900 2950 50  0001 C CNN
 	1    4900 2950
@@
 F 0 "sw_triggerAll1" H 3550 2400 50  0000 C CNN
 F 1 "SW_Push" H 3550 2644 50  0001 C CNN
-F 2 "" H 3550 2650 50  0001 C CNN
+F 2 "Button_Switch_THT:SW_PUSH_6mm" H 3550 2650 50  0001 C CNN
 F 3 "~" H 3550 2650 50  0001 C CNN
 	1    3550 2450
